File: pi-top_Template.kicad_pcb (KiCad board)
At the start: 2 copper layers, 65 x 56 mm, 6 parts, among them P1 CONN_17X2, P2 CONN_17X2

Commit message: Fix connector pin numbering
Parts:
- P1: value CONN_17X2 -> 3M_951_Series
- P2: value CONN_17X2 -> Harwin M22-655R; footprint Harwin_M22-655_Series -> Harwin_M22-655R
